File: Sheet1.sch (KiCad schematic (older format))
At the start: 52 parts, among them J1 Conn_01x02_Male, J2 Conn_01x02_Male, J3 Conn_01x02_Male, J4 Conn_01x02_Male, K1 G6S-2, K2 G6S-2, U1 TL074, U4 NE555, U5 NE555

Commit message: Resistors to SMD
Parts:
- R1, R10, R11, R12, R13, R14, R15, R16, R17, R18, R19, R2, R20, R3, R4, R5, R6, R7, R8, R9: footprint Resistor_THT:R_Axial_DIN0207_L6.3mm_D2.5mm_P7.62mm_Horizontal -> Resistor_SMD:R_0603_1608Metric
Connections:
- net GND: now also J1.1 (Pin_1), J2.1 (Pin_1); no longer J1.2 (Pin_2), J2.2 (Pin_2)
- net In: now also J1.2 (Pin_2); no longer J1.1 (Pin_1)
- net Out: now also J2.2 (Pin_2); no longer J2.1 (Pin_1)
- net at R14.2: now also RV1.3; no longer RV1.1
- net at R15.2: now also RV1.1; no longer RV1.3
Changed lines of the file:
@@
 F 0 "R4" V 3393 1750 50  0000 C CNN
 F 1 "100K" V 3484 1750 50  0000 C CNN
-F 2 "Resistor_THT:R_Axial_DIN0207_L6.3mm_D2.5mm_P7.62mm_Horizontal" V 3530 1750 50  0001 C CNN
+F 2 "Resistor_SMD:R_0603_1608Metric" V 3530 1750 50  0001 C CNN
 F 3 "~" H 3600 1750 50  0001 C CNN
 	1    3600 1750
@@
 F 0 "R6" V 3993 1400 50  0000 C CNN
 F 1 "100K" V 4084 1400 50  0000 C CNN
-F 2 "Resistor_THT:R_Axial_DIN0207_L6.3mm_D2.5mm_P7.62mm_Horizontal" V 4130 1400 50  0001 C CNN
+F 2 "Resistor_SMD:R_0603_1608Metric" V 4130 1400 50  0001 C CNN
 F 3 "~" H 4200 1400 50  0001 C CNN
 	1    4200 1400
@@
 F 0 "R7" V 3993 2650 50  0000 C CNN
 F 1 "100K" V 4084 2650 50  0000 C CNN
-F 2 "Resistor_THT:R_Axial_DIN0207_L6.3mm_D2.5mm_P7.62mm_Horizontal" V 4130 2650 50  0001 C CNN
+F 2 "Resistor_SMD:R_0603_1608Metric" V 4130 2650 50  0001 C CNN
 F 3 "~" H 4200 2650 50  0001 C CNN
 	1    4200 2650
@@
 F 0 "R3" H 3130 2004 50  0000 R CNN
 F 1 "500k" H 3130 2095 50  0000 R CNN
-F 2 "Resistor_THT:R_Axial_DIN0207_L6.3mm_D2.5mm_P7.62mm_Horizontal" V 3130 2050 50  0001 C CNN
+F 2 "Resistor_SMD:R_0603_1608Metric" V 3130 2050 50  0001 C CNN
 F 3 "~" H 3200 2050 50  0001 C CNN
 	1    3200 2050
@@
 F 0 "R5" V 3393 3000 50  0000 C CNN
 F 1 "100K" V 3484 3000 50  0000 C CNN
-F 2 "Resistor_THT:R_Axial_DIN0207_L6.3mm_D2.5mm_P7.62mm_Horizontal" V 3530 3000 50  0001 C CNN
+F 2 "Resistor_SMD:R_0603_1608Metric" V 3530 3000 50  0001 C CNN
 F 3 "~" H 3600 3000 50  0001 C CNN
 	1    3600 3000
@@
 F 0 "R13" H 6480 1804 50  0000 R CNN
 F 1 "10k" H 6480 1895 50  0000 R CNN
-F 2 "Resistor_THT:R_Axial_DIN0207_L6.3mm_D2.5mm_P7.62mm_Horizontal" V 6480 1850 50  0001 C CNN
+F 2 "Resistor_SMD:R_0603_1608Metric" V 6480 1850 50  0001 C CNN
 F 3 "~" H 6550 1850 50  0001 C CNN
 	1    6550 1850
@@
 F 0 "R17" H 7630 1054 50  0000 R CNN
 F 1 "10k" H 7630 1145 50  0000 R CNN
-F 2 "Resistor_THT:R_Axial_DIN0207_L6.3mm_D2.5mm_P7.62mm_Horizontal" V 7630 1100 50  0001 C CNN
+F 2 "Resistor_SMD:R_0603_1608Metric" V 7630 1100 50  0001 C CNN
 F 3 "~" H 7700 1100 50  0001 C CNN
 	1    7700 1100
@@
 F 0 "R18" H 8330 1204 50  0000 R CNN
 F 1 "4.7k" H 8330 1295 50  0000 R CNN
-F 2 "Resistor_THT:R_Axial_DIN0207_L6.3mm_D2.5mm_P7.62mm_Horizontal" V 8330 1250 50  0001 C CNN
+F 2 "Resistor_SMD:R_0603_1608Metric" V 8330 1250 50  0001 C CNN
 F 3 "~" H 8400 1250 50  0001 C CNN
 	1    8400 1250
@@
 F 0 "R20" H 9230 1904 50  0000 R CNN
 F 1 "100k" H 9230 1995 50  0000 R CNN
-F 2 "Resistor_THT:R_Axial_DIN0207_L6.3mm_D2.5mm_P7.62mm_Horizontal" V 9230 1950 50  0001 C CNN
+F 2 "Resistor_SMD:R_0603_1608Metric" V 9230 1950 50  0001 C CNN
 F 3 "~" H 9300 1950 50  0001 C CNN
 	1    9300 1950
@@
 F 0 "R14" H 6630 3104 50  0000 R CNN
 F 1 "100k" H 6630 3195 50  0000 R CNN
-F 2 "Resistor_THT:R_Axial_DIN0207_L6.3mm_D2.5mm_P7.62mm_Horizontal" V 6630 3150 50  0001 C CNN
+F 2 "Resistor_SMD:R_0603_1608Metric" V 6630 3150 50  0001 C CNN
 F 3 "~" H 6700 3150 50  0001 C CNN
 	1    6700 3150
@@
 F 0 "R15" H 6630 3554 50  0000 R CNN
 F 1 "100k" H 6630 3645 50  0000 R CNN
-F 2 "Resistor_THT:R_Axial_DIN0207_L6.3mm_D2.5mm_P7.62mm_Horizontal" V 6630 3600 50  0001 C CNN
+F 2 "Resistor_SMD:R_0603_1608Metric" V 6630 3600 50  0001 C CNN
 F 3 "~" H 6700 3600 50  0001 C CNN
 	1    6700 3600
 	0    -1   -1   0
-$EndComp
-$Comp
-L Device:R_POT RV1
-U 1 1 61308C3E
-P 7050 3400
-F 0 "RV1" H 6981 3446 50  0000 R CNN
-F 1 "B100k" H 6981 3355 50  0000 R CNN
-F 2 "MBv3 potentiometers:16MM_B.MOUNT_BANZAI" H 7050 3400 50  0001 C CNN
-F 3 "~" H 7050 3400 50  0001 C CNN
-	1    7050 3400
-	1    0    0    -1
 $EndComp
 Wire Wire Line
@@
 F 0 "R16" H 7580 2754 50  0000 R CNN
 F 1 "100k" H 7580 2845 50  0000 R CNN
-F 2 "Resistor_THT:R_Axial_DIN0207_L6.3mm_D2.5mm_P7.62mm_Horizontal" V 7580 2800 50  0001 C CNN
+F 2 "Resistor_SMD:R_0603_1608Metric" V 7580 2800 50  0001 C CNN
 F 3 "~" H 7650 2800 50  0001 C CNN
 	1    7650 2800
@@
 F 0 "R19" H 8380 3454 50  0000 R CNN
 F 1 "1k" H 8380 3545 50  0000 R CNN
-F 2 "Resistor_THT:R_Axial_DIN0207_L6.3mm_D2.5mm_P7.62mm_Horizontal" V 8380 3500 50  0001 C CNN
+F 2 "Resistor_SMD:R_0603_1608Metric" V 8380 3500 50  0001 C CNN
 F 3 "~" H 8450 3500 50  0001 C CNN
 	1    8450 3500
@@
 F 0 "R1" H 2680 2054 50  0000 R CNN
 F 1 "500k" H 2680 2145 50  0000 R CNN
-F 2 "Resistor_THT:R_Axial_DIN0207_L6.3mm_D2.5mm_P7.62mm_Horizontal" V 2680 2100 50  0001 C CNN
+F 2 "Resistor_SMD:R_0603_1608Metric" V 2680 2100 50  0001 C CNN
 F 3 "~" H 2750 2100 50  0001 C CNN
 	1    2750 2100
@@
 F 0 "R10" V 4693 5850 50  0000 C CNN
 F 1 "100K" V 4784 5850 50  0000 C CNN
-F 2 "Resistor_THT:R_Axial_DIN0207_L6.3mm_D2.5mm_P7.62mm_Horizontal" V 4830 5850 50  0001 C CNN
+F 2 "Resistor_SMD:R_0603_1608Metric" V 4830 5850 50  0001 C CNN
 F 3 "~" H 4900 5850 50  0001 C CNN
 	1    4900 5850
@@
 F 0 "R12" V 6293 4800 50  0000 C CNN
 F 1 "4.7k" V 6384 4800 50  0000 C CNN
-F 2 "Resistor_THT:R_Axial_DIN0207_L6.3mm_D2.5mm_P7.62mm_Horizontal" V 6430 4800 50  0001 C CNN
+F 2 "Resistor_SMD:R_0603_1608Metric" V 6430 4800 50  0001 C CNN
 F 3 "~" H 6500 4800 50  0001 C CNN
 	1    6500 4800
@@
 F 0 "R9" V 2893 4800 50  0000 C CNN
 F 1 "4.7k" V 2984 4800 50  0000 C CNN
-F 2 "Resistor_THT:R_Axial_DIN0207_L6.3mm_D2.5mm_P7.62mm_Horizontal" V 3030 4800 50  0001 C CNN
+F 2 "Resistor_SMD:R_0603_1608Metric" V 3030 4800 50  0001 C CNN
 F 3 "~" H 3100 4800 50  0001 C CNN
 	1    3100 4800
@@
 F 0 "R2" V 1143 5850 50  0000 C CNN
 F 1 "100K" V 1234 5850 50  0000 C CNN
-F 2 "Resistor_THT:R_Axial_DIN0207_L6.3mm_D2.5mm_P7.62mm_Horizontal" V 1280 5850 50  0001 C CNN
+F 2 "Resistor_SMD:R_0603_1608Metric" V 1280 5850 50  0001 C CNN
 F 3 "~" H 1350 5850 50  0001 C CNN
 	1    1350 5850
@@
 F 0 "R8" V 2693 5200 50  0000 C CNN
 F 1 "10k" V 2784 5200 50  0000 C CNN
-F 2 "Resistor_THT:R_Axial_DIN0207_L6.3mm_D2.5mm_P7.62mm_Horizontal" V 2830 5200 50  0001 C CNN
+F 2 "Resistor_SMD:R_0603_1608Metric" V 2830 5200 50  0001 C CNN
 F 3 "~" H 2900 5200 50  0001 C CNN
 	1    2900 5200
@@
 F 0 "R11" V 6143 5200 50  0000 C CNN
 F 1 "10k" V 6234 5200 50  0000 C CNN
-F 2 "Resistor_THT:R_Axial_DIN0207_L6.3mm_D2.5mm_P7.62mm_Horizontal" V 6280 5200 50  0001 C CNN
+F 2 "Resistor_SMD:R_0603_1608Metric" V 6280 5200 50  0001 C CNN
 F 3 "~" H 6350 5200 50  0001 C CNN
 	1    6350 5200
@@
 	2100 7200 2200 7200
 Connection ~ 2200 7200
-Text GLabel 1250 950  2    50   Input ~ 0
+Text GLabel 1250 1050 2    50   Input ~ 0
 In
-Wire Wire Line
-	900  950  1250 950
 Wire Wire Line
 	900  1050 1250 1050
@@
 L power:GND #PWR0166
 U 1 1 617CF781
-P 1250 1050
-F 0 "#PWR0166" H 1250 800 50  0001 C CNN
-F 1 "GND" H 1255 877 50  0000 C CNN
-F 2 "" H 1250 1050 50  0001 C CNN
-F 3 "" H 1250 1050 50  0001 C CNN
-	1    1250 1050
-	1    0    0    -1
-$EndComp
-Text GLabel 1250 1400 2    50   Input ~ 0
+P 1550 950
+F 0 "#PWR0166" H 1550 700 50  0001 C CNN
+F 1 "GND" H 1555 777 50  0000 C CNN
+F 2 "" H 1550 950 50  0001 C CNN
+F 3 "" H 1550 950 50  0001 C CNN
+	1    1550 950
+	1    0    0    -1
+$EndComp
+Text GLabel 1250 1500 2    50   Input ~ 0
 Out
-Wire Wire Line
-	1250 1400 900  1400
 $Comp
 L power:GND #PWR0167
 U 1 1 617D802A
-P 1250 1500
-F 0 "#PWR0167" H 1250 1250 50  0001 C CNN
-F 1 "GND" H 1255 1327 50  0000 C CNN
-F 2 "" H 1250 1500 50  0001 C CNN
-F 3 "" H 1250 1500 50  0001 C CNN
-	1    1250 1500
+P 1550 1400
+F 0 "#PWR0167" H 1550 1150 50  0001 C CNN
+F 1 "GND" H 1555 1227 50  0000 C CNN
+F 2 "" H 1550 1400 50  0001 C CNN
+F 3 "" H 1550 1400 50  0001 C CNN
+	1    1550 1400
 	1    0    0    -1
 $EndComp
@@
 Wire Wire Line
 	8700 3500 8850 3500
+$Comp
+L Device:R_POT RV1
+U 1 1 61308C3E
+P 7050 3400
+F 0 "RV1" H 6981 3446 50  0000 R CNN
+F 1 "B100k" H 6981 3355 50  0000 R CNN
+F 2 "MBv3 potentiometers:16MM_B.MOUNT_BANZAI" H 7050 3400 50  0001 C CNN
+F 3 "~" H 7050 3400 50  0001 C CNN
+	1    7050 3400
+	1    0    0    1
+$EndComp
+Wire Wire Line
+	900  950  1550 950
+Wire Wire Line
+	900  1400 1550 1400
 $EndSCHEMATC

Commit message: 2 layer dead end
Parts:
- added Q3: J201, Package_TO_SOT_THT:TO-92L_Inline_Wide, symbol Device:Q_NJFET_DSG
- added R41: 20k, Resistor_SMD:R_0603_1608Metric, symbol Device:R
- C3, C4: value 5p -> 1p
- R1: value 500k -> 1M
- R3: value 500k -> 200k
- R4, R5, R6, R7: value 100K -> 10k
Connections:
- net +9V: now also Q3.1 (D)
- net -9V: now also R41.1
- net EffectIn: now also Q3.3 (G); no longer C2.2
- new net: C2.2, Q3.2 (S), R41.2
Other:
- moved on the sheet: C2, J1, J2, J3, J4, R1, R3

Commit message: v1 sent to JLC
Parts:
- R1, R10, R11, R12, R13, R14, R15, R16, R17, R18, R19, R2, R20, R3, R4, R41, R5, R6, R7, R8, R9: footprint Resistor_SMD:R_0603_1608Metric -> Resistor_SMD:R_0603_1608Metric_Pad1.05x0.95mm_HandSolder
Changed lines of the file:
@@
 encoding utf-8
 Sheet 2 4
-Title ""
-Date ""
-Rev ""
-Comp ""
+Title "Ping"
+Date "2021-08-31"
+Rev "1"
+Comp "Andrei Salomatin"
 Comment1 ""
 Comment2 ""
@@
 F 0 "R4" V 3393 1750 50  0000 C CNN
 F 1 "10k" V 3484 1750 50  0000 C CNN
-F 2 "Resistor_SMD:R_0603_1608Metric" V 3530 1750 50  0001 C CNN
+F 2 "Resistor_SMD:R_0603_1608Metric_Pad1.05x0.95mm_HandSolder" V 3530 1750 50  0001 C CNN
 F 3 "~" H 3600 1750 50  0001 C CNN
 	1    3600 1750
@@
 F 0 "R6" V 3993 1400 50  0000 C CNN
 F 1 "10k" V 4084 1400 50  0000 C CNN
-F 2 "Resistor_SMD:R_0603_1608Metric" V 4130 1400 50  0001 C CNN
+F 2 "Resistor_SMD:R_0603_1608Metric_Pad1.05x0.95mm_HandSolder" V 4130 1400 50  0001 C CNN
 F 3 "~" H 4200 1400 50  0001 C CNN
 	1    4200 1400
@@
 F 0 "R7" V 3993 2650 50  0000 C CNN
 F 1 "10k" V 4084 2650 50  0000 C CNN
-F 2 "Resistor_SMD:R_0603_1608Metric" V 4130 2650 50  0001 C CNN
+F 2 "Resistor_SMD:R_0603_1608Metric_Pad1.05x0.95mm_HandSolder" V 4130 2650 50  0001 C CNN
 F 3 "~" H 4200 2650 50  0001 C CNN
 	1    4200 2650
@@
 F 0 "R3" H 3030 2004 50  0000 R CNN
 F 1 "200k" H 3030 2095 50  0000 R CNN
-F 2 "Resistor_SMD:R_0603_1608Metric" V 3030 2050 50  0001 C CNN
+F 2 "Resistor_SMD:R_0603_1608Metric_Pad1.05x0.95mm_HandSolder" V 3030 2050 50  0001 C CNN
 F 3 "~" H 3100 2050 50  0001 C CNN
 	1    3100 2050
@@
 F 0 "R5" V 3393 3000 50  0000 C CNN
 F 1 "10k" V 3484 3000 50  0000 C CNN
-F 2 "Resistor_SMD:R_0603_1608Metric" V 3530 3000 50  0001 C CNN
+F 2 "Resistor_SMD:R_0603_1608Metric_Pad1.05x0.95mm_HandSolder" V 3530 3000 50  0001 C CNN
 F 3 "~" H 3600 3000 50  0001 C CNN
 	1    3600 3000
@@
 F 0 "R13" H 6480 1804 50  0000 R CNN
 F 1 "10k" H 6480 1895 50  0000 R CNN
-F 2 "Resistor_SMD:R_0603_1608Metric" V 6480 1850 50  0001 C CNN
+F 2 "Resistor_SMD:R_0603_1608Metric_Pad1.05x0.95mm_HandSolder" V 6480 1850 50  0001 C CNN
 F 3 "~" H 6550 1850 50  0001 C CNN
 	1    6550 1850
@@
 F 0 "R17" H 7630 1054 50  0000 R CNN
 F 1 "10k" H 7630 1145 50  0000 R CNN
-F 2 "Resistor_SMD:R_0603_1608Metric" V 7630 1100 50  0001 C CNN
+F 2 "Resistor_SMD:R_0603_1608Metric_Pad1.05x0.95mm_HandSolder" V 7630 1100 50  0001 C CNN
 F 3 "~" H 7700 1100 50  0001 C CNN
 	1    7700 1100
@@
 F 0 "R18" H 8330 1204 50  0000 R CNN
 F 1 "4.7k" H 8330 1295 50  0000 R CNN
-F 2 "Resistor_SMD:R_0603_1608Metric" V 8330 1250 50  0001 C CNN
+F 2 "Resistor_SMD:R_0603_1608Metric_Pad1.05x0.95mm_HandSolder" V 8330 1250 50  0001 C CNN
 F 3 "~" H 8400 1250 50  0001 C CNN
 	1    8400 1250
@@
 F 0 "R20" H 9230 1904 50  0000 R CNN
 F 1 "100k" H 9230 1995 50  0000 R CNN
-F 2 "Resistor_SMD:R_0603_1608Metric" V 9230 1950 50  0001 C CNN
+F 2 "Resistor_SMD:R_0603_1608Metric_Pad1.05x0.95mm_HandSolder" V 9230 1950 50  0001 C CNN
 F 3 "~" H 9300 1950 50  0001 C CNN
 	1    9300 1950
@@
 F 0 "R14" H 6630 3104 50  0000 R CNN
 F 1 "100k" H 6630 3195 50  0000 R CNN
-F 2 "Resistor_SMD:R_0603_1608Metric" V 6630 3150 50  0001 C CNN
+F 2 "Resistor_SMD:R_0603_1608Metric_Pad1.05x0.95mm_HandSolder" V 6630 3150 50  0001 C CNN
 F 3 "~" H 6700 3150 50  0001 C CNN
 	1    6700 3150
@@
 F 0 "R15" H 6630 3554 50  0000 R CNN
 F 1 "100k" H 6630 3645 50  0000 R CNN
-F 2 "Resistor_SMD:R_0603_1608Metric" V 6630 3600 50  0001 C CNN
+F 2 "Resistor_SMD:R_0603_1608Metric_Pad1.05x0.95mm_HandSolder" V 6630 3600 50  0001 C CNN
 F 3 "~" H 6700 3600 50  0001 C CNN
 	1    6700 3600
@@
 F 0 "R16" H 7580 2754 50  0000 R CNN
 F 1 "100k" H 7580 2845 50  0000 R CNN
-F 2 "Resistor_SMD:R_0603_1608Metric" V 7580 2800 50  0001 C CNN
+F 2 "Resistor_SMD:R_0603_1608Metric_Pad1.05x0.95mm_HandSolder" V 7580 2800 50  0001 C CNN
 F 3 "~" H 7650 2800 50  0001 C CNN
 	1    7650 2800
@@
 F 0 "R19" H 8380 3454 50  0000 R CNN
 F 1 "1k" H 8380 3545 50  0000 R CNN
-F 2 "Resistor_SMD:R_0603_1608Metric" V 8380 3500 50  0001 C CNN
+F 2 "Resistor_SMD:R_0603_1608Metric_Pad1.05x0.95mm_HandSolder" V 8380 3500 50  0001 C CNN
 F 3 "~" H 8450 3500 50  0001 C CNN
 	1    8450 3500
@@
 F 0 "R1" H 1880 1704 50  0000 R CNN
 F 1 "1M" H 1880 1795 50  0000 R CNN
-F 2 "Resistor_SMD:R_0603_1608Metric" V 1880 1750 50  0001 C CNN
+F 2 "Resistor_SMD:R_0603_1608Metric_Pad1.05x0.95mm_HandSolder" V 1880 1750 50  0001 C CNN
 F 3 "~" H 1950 1750 50  0001 C CNN
 	1    1950 1750
@@
 F 0 "R10" V 4693 5850 50  0000 C CNN
 F 1 "100K" V 4784 5850 50  0000 C CNN
-F 2 "Resistor_SMD:R_0603_1608Metric" V 4830 5850 50  0001 C CNN
+F 2 "Resistor_SMD:R_0603_1608Metric_Pad1.05x0.95mm_HandSolder" V 4830 5850 50  0001 C CNN
 F 3 "~" H 4900 5850 50  0001 C CNN
 	1    4900 5850
@@
 F 0 "R12" V 6293 4800 50  0000 C CNN
 F 1 "4.7k" V 6384 4800 50  0000 C CNN
-F 2 "Resistor_SMD:R_0603_1608Metric" V 6430 4800 50  0001 C CNN
+F 2 "Resistor_SMD:R_0603_1608Metric_Pad1.05x0.95mm_HandSolder" V 6430 4800 50  0001 C CNN
 F 3 "~" H 6500 4800 50  0001 C CNN
 	1    6500 4800
@@
 F 0 "R9" V 2893 4800 50  0000 C CNN
 F 1 "4.7k" V 2984 4800 50  0000 C CNN
-F 2 "Resistor_SMD:R_0603_1608Metric" V 3030 4800 50  0001 C CNN
+F 2 "Resistor_SMD:R_0603_1608Metric_Pad1.05x0.95mm_HandSolder" V 3030 4800 50  0001 C CNN
 F 3 "~" H 3100 4800 50  0001 C CNN
 	1    3100 4800
@@
 F 0 "R2" V 1143 5850 50  0000 C CNN
 F 1 "100K" V 1234 5850 50  0000 C CNN
-F 2 "Resistor_SMD:R_0603_1608Metric" V 1280 5850 50  0001 C CNN
+F 2 "Resistor_SMD:R_0603_1608Metric_Pad1.05x0.95mm_HandSolder" V 1280 5850 50  0001 C CNN
 F 3 "~" H 1350 5850 50  0001 C CNN
 	1    1350 5850
@@
 F 0 "R8" V 2693 5200 50  0000 C CNN
 F 1 "10k" V 2784 5200 50  0000 C CNN
-F 2 "Resistor_SMD:R_0603_1608Metric" V 2830 5200 50  0001 C CNN
+F 2 "Resistor_SMD:R_0603_1608Metric_Pad1.05x0.95mm_HandSolder" V 2830 5200 50  0001 C CNN
 F 3 "~" H 2900 5200 50  0001 C CNN
 	1    2900 5200
@@
 F 0 "R11" V 6143 5200 50  0000 C CNN
 F 1 "10k" V 6234 5200 50  0000 C CNN
-F 2 "Resistor_SMD:R_0603_1608Metric" V 6280 5200 50  0001 C CNN
+F 2 "Resistor_SMD:R_0603_1608Metric_Pad1.05x0.95mm_HandSolder" V 6280 5200 50  0001 C CNN
 F 3 "~" H 6350 5200 50  0001 C CNN
 	1    6350 5200
@@
 F 0 "R41" H 2330 1904 50  0000 R CNN
 F 1 "20k" H 2330 1995 50  0000 R CNN
-F 2 "Resistor_SMD:R_0603_1608Metric" V 2330 1950 50  0001 C CNN
+F 2 "Resistor_SMD:R_0603_1608Metric_Pad1.05x0.95mm_HandSolder" V 2330 1950 50  0001 C CNN
 F 3 "~" H 2400 1950 50  0001 C CNN
 	1    2400 1950
