File: Sheet2.sch (KiCad schematic (older format))
At the start: 44 parts, among them IC1 BTDR-3, J5 Conn_01x04_Male, Q1 BC558C, Q2 BC558C, U2 TL074, U3 LM13700

Commit message: Resistors to SMD
Parts:
- R21, R22, R23, R24, R25, R26, R27, R28, R29, R30, R31, R32, R33, R34, R35, R36, R37, R38, R39, R40: footprint Resistor_THT:R_Axial_DIN0207_L6.3mm_D2.5mm_P7.62mm_Horizontal -> Resistor_SMD:R_0603_1608Metric
Connections:
- net FilterOut: now also RV3.3; no longer RV3.1
- net FreqCV: now also RV2.3; no longer RV2.1
- net GND: now also RV2.1, RV3.1; no longer RV2.3, RV3.3
Changed lines of the file:
@@
 F 0 "R22" V 1143 3750 50  0000 C CNN
 F 1 "10k" V 1234 3750 50  0000 C CNN
-F 2 "Resistor_THT:R_Axial_DIN0207_L6.3mm_D2.5mm_P7.62mm_Horizontal" V 1280 3750 50  0001 C CNN
+F 2 "Resistor_SMD:R_0603_1608Metric" V 1280 3750 50  0001 C CNN
 F 3 "~" H 1350 3750 50  0001 C CNN
 	1    1350 3750
@@
 F 0 "R23" H 1630 4104 50  0000 R CNN
 F 1 "220" H 1630 4195 50  0000 R CNN
-F 2 "Resistor_THT:R_Axial_DIN0207_L6.3mm_D2.5mm_P7.62mm_Horizontal" V 1630 4150 50  0001 C CNN
+F 2 "Resistor_SMD:R_0603_1608Metric" V 1630 4150 50  0001 C CNN
 F 3 "~" H 1700 4150 50  0001 C CNN
 	1    1700 4150
@@
 F 0 "R25" H 2330 4104 50  0000 R CNN
 F 1 "220" H 2330 4195 50  0000 R CNN
-F 2 "Resistor_THT:R_Axial_DIN0207_L6.3mm_D2.5mm_P7.62mm_Horizontal" V 2330 4150 50  0001 C CNN
+F 2 "Resistor_SMD:R_0603_1608Metric" V 2330 4150 50  0001 C CNN
 F 3 "~" H 2400 4150 50  0001 C CNN
 	1    2400 4150
@@
 F 0 "R24" V 2357 4000 50  0000 C CNN
 F 1 "10k" V 2266 4000 50  0000 C CNN
-F 2 "Resistor_THT:R_Axial_DIN0207_L6.3mm_D2.5mm_P7.62mm_Horizontal" V 2080 4000 50  0001 C CNN
+F 2 "Resistor_SMD:R_0603_1608Metric" V 2080 4000 50  0001 C CNN
 F 3 "~" H 2150 4000 50  0001 C CNN
 	1    2150 4000
@@
 F 0 "R29" H 3180 4104 50  0000 R CNN
 F 1 "10k" H 3180 4195 50  0000 R CNN
-F 2 "Resistor_THT:R_Axial_DIN0207_L6.3mm_D2.5mm_P7.62mm_Horizontal" V 3180 4150 50  0001 C CNN
+F 2 "Resistor_SMD:R_0603_1608Metric" V 3180 4150 50  0001 C CNN
 F 3 "~" H 3250 4150 50  0001 C CNN
 	1    3250 4150
@@
 F 0 "R27" H 2880 3054 50  0000 R CNN
 F 1 "10k" H 2880 3145 50  0000 R CNN
-F 2 "Resistor_THT:R_Axial_DIN0207_L6.3mm_D2.5mm_P7.62mm_Horizontal" V 2880 3100 50  0001 C CNN
+F 2 "Resistor_SMD:R_0603_1608Metric" V 2880 3100 50  0001 C CNN
 F 3 "~" H 2950 3100 50  0001 C CNN
 	1    2950 3100
@@
 F 0 "R34" H 4730 3704 50  0000 R CNN
 F 1 "10k" H 4730 3795 50  0000 R CNN
-F 2 "Resistor_THT:R_Axial_DIN0207_L6.3mm_D2.5mm_P7.62mm_Horizontal" V 4730 3750 50  0001 C CNN
+F 2 "Resistor_SMD:R_0603_1608Metric" V 4730 3750 50  0001 C CNN
 F 3 "~" H 4800 3750 50  0001 C CNN
 	1    4800 3750
@@
 F 0 "R35" H 4980 4054 50  0000 R CNN
 F 1 "220" H 4980 4145 50  0000 R CNN
-F 2 "Resistor_THT:R_Axial_DIN0207_L6.3mm_D2.5mm_P7.62mm_Horizontal" V 4980 4100 50  0001 C CNN
+F 2 "Resistor_SMD:R_0603_1608Metric" V 4980 4100 50  0001 C CNN
 F 3 "~" H 5050 4100 50  0001 C CNN
 	1    5050 4100
@@
 F 0 "R37" H 5280 4054 50  0000 R CNN
 F 1 "220" H 5280 4145 50  0000 R CNN
-F 2 "Resistor_THT:R_Axial_DIN0207_L6.3mm_D2.5mm_P7.62mm_Horizontal" V 5280 4100 50  0001 C CNN
+F 2 "Resistor_SMD:R_0603_1608Metric" V 5280 4100 50  0001 C CNN
 F 3 "~" H 5350 4100 50  0001 C CNN
 	1    5350 4100
@@
 F 0 "R36" V 5557 3400 50  0000 C CNN
 F 1 "10k" V 5466 3400 50  0000 C CNN
-F 2 "Resistor_THT:R_Axial_DIN0207_L6.3mm_D2.5mm_P7.62mm_Horizontal" V 5280 3400 50  0001 C CNN
+F 2 "Resistor_SMD:R_0603_1608Metric" V 5280 3400 50  0001 C CNN
 F 3 "~" H 5350 3400 50  0001 C CNN
 	1    5350 3400
@@
 F 0 "R38" H 6080 3954 50  0000 R CNN
 F 1 "10k" H 6080 4045 50  0000 R CNN
-F 2 "Resistor_THT:R_Axial_DIN0207_L6.3mm_D2.5mm_P7.62mm_Horizontal" V 6080 4000 50  0001 C CNN
+F 2 "Resistor_SMD:R_0603_1608Metric" V 6080 4000 50  0001 C CNN
 F 3 "~" H 6150 4000 50  0001 C CNN
 	1    6150 4000
@@
 F 0 "R39" H 6180 2804 50  0000 R CNN
 F 1 "10k" H 6180 2895 50  0000 R CNN
-F 2 "Resistor_THT:R_Axial_DIN0207_L6.3mm_D2.5mm_P7.62mm_Horizontal" V 6180 2850 50  0001 C CNN
+F 2 "Resistor_SMD:R_0603_1608Metric" V 6180 2850 50  0001 C CNN
 F 3 "~" H 6250 2850 50  0001 C CNN
 	1    6250 2850
@@
 F 3 "~" H 8150 3900 50  0001 C CNN
 	1    8150 3900
-	-1   0    0    -1
+	-1   0    0    1
 $EndComp
 Wire Wire Line
@@
 F 0 "R31" V 4257 4950 50  0000 C CNN
 F 1 "10k" V 4166 4950 50  0000 C CNN
-F 2 "Resistor_THT:R_Axial_DIN0207_L6.3mm_D2.5mm_P7.62mm_Horizontal" V 3980 4950 50  0001 C CNN
+F 2 "Resistor_SMD:R_0603_1608Metric" V 3980 4950 50  0001 C CNN
 F 3 "~" H 4050 4950 50  0001 C CNN
 	1    4050 4950
@@
 F 0 "R32" H 4480 5704 50  0000 R CNN
 F 1 "1.6K" H 4480 5795 50  0000 R CNN
-F 2 "Resistor_THT:R_Axial_DIN0207_L6.3mm_D2.5mm_P7.62mm_Horizontal" V 4480 5750 50  0001 C CNN
+F 2 "Resistor_SMD:R_0603_1608Metric" V 4480 5750 50  0001 C CNN
 F 3 "~" H 4550 5750 50  0001 C CNN
 	1    4550 5750
@@
 F 0 "R33" V 4493 1000 50  0000 C CNN
 F 1 "4.7k" V 4584 1000 50  0000 C CNN
-F 2 "Resistor_THT:R_Axial_DIN0207_L6.3mm_D2.5mm_P7.62mm_Horizontal" V 4630 1000 50  0001 C CNN
+F 2 "Resistor_SMD:R_0603_1608Metric" V 4630 1000 50  0001 C CNN
 F 3 "~" H 4700 1000 50  0001 C CNN
 	1    4700 1000
@@
 F 0 "R30" H 3630 2004 50  0000 R CNN
 F 1 "470k" H 3630 2095 50  0000 R CNN
-F 2 "Resistor_THT:R_Axial_DIN0207_L6.3mm_D2.5mm_P7.62mm_Horizontal" V 3630 2050 50  0001 C CNN
+F 2 "Resistor_SMD:R_0603_1608Metric" V 3630 2050 50  0001 C CNN
 F 3 "~" H 3700 2050 50  0001 C CNN
 	1    3700 2050
@@
 F 0 "R28" H 3030 2004 50  0000 R CNN
 F 1 "2.7k" H 3030 2095 50  0000 R CNN
-F 2 "Resistor_THT:R_Axial_DIN0207_L6.3mm_D2.5mm_P7.62mm_Horizontal" V 3030 2050 50  0001 C CNN
+F 2 "Resistor_SMD:R_0603_1608Metric" V 3030 2050 50  0001 C CNN
 F 3 "~" H 3100 2050 50  0001 C CNN
 	1    3100 2050
@@
 F 0 "R26" V 2543 1500 50  0000 C CNN
 F 1 "100k" V 2634 1500 50  0000 C CNN
-F 2 "Resistor_THT:R_Axial_DIN0207_L6.3mm_D2.5mm_P7.62mm_Horizontal" V 2680 1500 50  0001 C CNN
+F 2 "Resistor_SMD:R_0603_1608Metric" V 2680 1500 50  0001 C CNN
 F 3 "~" H 2750 1500 50  0001 C CNN
 	1    2750 1500
@@
 F 0 "R40" H 10080 1754 50  0000 R CNN
 F 1 "100k" H 10080 1845 50  0000 R CNN
-F 2 "Resistor_THT:R_Axial_DIN0207_L6.3mm_D2.5mm_P7.62mm_Horizontal" V 10080 1800 50  0001 C CNN
+F 2 "Resistor_SMD:R_0603_1608Metric" V 10080 1800 50  0001 C CNN
 F 3 "~" H 10150 1800 50  0001 C CNN
 	1    10150 1800
@@
 F 3 "~" H 2250 1500 50  0001 C CNN
 	1    2250 1500
-	1    0    0    -1
+	1    0    0    1
 $EndComp
 $Comp
@@
 F 0 "R21" V 1293 1500 50  0000 C CNN
 F 1 "100" V 1384 1500 50  0000 C CNN
-F 2 "Resistor_THT:R_Axial_DIN0207_L6.3mm_D2.5mm_P7.62mm_Horizontal" V 1430 1500 50  0001 C CNN
+F 2 "Resistor_SMD:R_0603_1608Metric" V 1430 1500 50  0001 C CNN
 F 3 "~" H 1500 1500 50  0001 C CNN
 	1    1500 1500

Commit message: v1 sent to JLC
Parts:
- R21, R22, R23, R24, R25, R26, R27, R28, R29, R30, R31, R32, R33, R34, R35, R36, R37, R38, R39, R40: footprint Resistor_SMD:R_0603_1608Metric -> Resistor_SMD:R_0603_1608Metric_Pad1.05x0.95mm_HandSolder
Changed lines of the file:
@@
 encoding utf-8
 Sheet 3 4
-Title ""
-Date ""
-Rev ""
-Comp ""
+Title "Ping"
+Date "2021-08-31"
+Rev "1"
+Comp "Andrei Salomatin"
 Comment1 ""
 Comment2 ""
@@
 F 0 "R22" V 1143 3750 50  0000 C CNN
 F 1 "10k" V 1234 3750 50  0000 C CNN
-F 2 "Resistor_SMD:R_0603_1608Metric" V 1280 3750 50  0001 C CNN
+F 2 "Resistor_SMD:R_0603_1608Metric_Pad1.05x0.95mm_HandSolder" V 1280 3750 50  0001 C CNN
 F 3 "~" H 1350 3750 50  0001 C CNN
 	1    1350 3750
@@
 F 0 "R23" H 1630 4104 50  0000 R CNN
 F 1 "220" H 1630 4195 50  0000 R CNN
-F 2 "Resistor_SMD:R_0603_1608Metric" V 1630 4150 50  0001 C CNN
+F 2 "Resistor_SMD:R_0603_1608Metric_Pad1.05x0.95mm_HandSolder" V 1630 4150 50  0001 C CNN
 F 3 "~" H 1700 4150 50  0001 C CNN
 	1    1700 4150
@@
 F 0 "R25" H 2330 4104 50  0000 R CNN
 F 1 "220" H 2330 4195 50  0000 R CNN
-F 2 "Resistor_SMD:R_0603_1608Metric" V 2330 4150 50  0001 C CNN
+F 2 "Resistor_SMD:R_0603_1608Metric_Pad1.05x0.95mm_HandSolder" V 2330 4150 50  0001 C CNN
 F 3 "~" H 2400 4150 50  0001 C CNN
 	1    2400 4150
@@
 F 0 "R24" V 2357 4000 50  0000 C CNN
 F 1 "10k" V 2266 4000 50  0000 C CNN
-F 2 "Resistor_SMD:R_0603_1608Metric" V 2080 4000 50  0001 C CNN
+F 2 "Resistor_SMD:R_0603_1608Metric_Pad1.05x0.95mm_HandSolder" V 2080 4000 50  0001 C CNN
 F 3 "~" H 2150 4000 50  0001 C CNN
 	1    2150 4000
@@
 F 0 "R29" H 3180 4104 50  0000 R CNN
 F 1 "10k" H 3180 4195 50  0000 R CNN
-F 2 "Resistor_SMD:R_0603_1608Metric" V 3180 4150 50  0001 C CNN
+F 2 "Resistor_SMD:R_0603_1608Metric_Pad1.05x0.95mm_HandSolder" V 3180 4150 50  0001 C CNN
 F 3 "~" H 3250 4150 50  0001 C CNN
 	1    3250 4150
@@
 F 0 "R27" H 2880 3054 50  0000 R CNN
 F 1 "10k" H 2880 3145 50  0000 R CNN
-F 2 "Resistor_SMD:R_0603_1608Metric" V 2880 3100 50  0001 C CNN
+F 2 "Resistor_SMD:R_0603_1608Metric_Pad1.05x0.95mm_HandSolder" V 2880 3100 50  0001 C CNN
 F 3 "~" H 2950 3100 50  0001 C CNN
 	1    2950 3100
@@
 F 0 "R34" H 4730 3704 50  0000 R CNN
 F 1 "10k" H 4730 3795 50  0000 R CNN
-F 2 "Resistor_SMD:R_0603_1608Metric" V 4730 3750 50  0001 C CNN
+F 2 "Resistor_SMD:R_0603_1608Metric_Pad1.05x0.95mm_HandSolder" V 4730 3750 50  0001 C CNN
 F 3 "~" H 4800 3750 50  0001 C CNN
 	1    4800 3750
@@
 F 0 "R35" H 4980 4054 50  0000 R CNN
 F 1 "220" H 4980 4145 50  0000 R CNN
-F 2 "Resistor_SMD:R_0603_1608Metric" V 4980 4100 50  0001 C CNN
+F 2 "Resistor_SMD:R_0603_1608Metric_Pad1.05x0.95mm_HandSolder" V 4980 4100 50  0001 C CNN
 F 3 "~" H 5050 4100 50  0001 C CNN
 	1    5050 4100
@@
 F 0 "R37" H 5280 4054 50  0000 R CNN
 F 1 "220" H 5280 4145 50  0000 R CNN
-F 2 "Resistor_SMD:R_0603_1608Metric" V 5280 4100 50  0001 C CNN
+F 2 "Resistor_SMD:R_0603_1608Metric_Pad1.05x0.95mm_HandSolder" V 5280 4100 50  0001 C CNN
 F 3 "~" H 5350 4100 50  0001 C CNN
 	1    5350 4100
@@
 F 0 "R36" V 5557 3400 50  0000 C CNN
 F 1 "10k" V 5466 3400 50  0000 C CNN
-F 2 "Resistor_SMD:R_0603_1608Metric" V 5280 3400 50  0001 C CNN
+F 2 "Resistor_SMD:R_0603_1608Metric_Pad1.05x0.95mm_HandSolder" V 5280 3400 50  0001 C CNN
 F 3 "~" H 5350 3400 50  0001 C CNN
 	1    5350 3400
@@
 F 0 "R38" H 6080 3954 50  0000 R CNN
 F 1 "10k" H 6080 4045 50  0000 R CNN
-F 2 "Resistor_SMD:R_0603_1608Metric" V 6080 4000 50  0001 C CNN
+F 2 "Resistor_SMD:R_0603_1608Metric_Pad1.05x0.95mm_HandSolder" V 6080 4000 50  0001 C CNN
 F 3 "~" H 6150 4000 50  0001 C CNN
 	1    6150 4000
@@
 F 0 "R39" H 6180 2804 50  0000 R CNN
 F 1 "10k" H 6180 2895 50  0000 R CNN
-F 2 "Resistor_SMD:R_0603_1608Metric" V 6180 2850 50  0001 C CNN
+F 2 "Resistor_SMD:R_0603_1608Metric_Pad1.05x0.95mm_HandSolder" V 6180 2850 50  0001 C CNN
 F 3 "~" H 6250 2850 50  0001 C CNN
 	1    6250 2850
@@
 F 0 "R31" V 4257 4950 50  0000 C CNN
 F 1 "10k" V 4166 4950 50  0000 C CNN
-F 2 "Resistor_SMD:R_0603_1608Metric" V 3980 4950 50  0001 C CNN
+F 2 "Resistor_SMD:R_0603_1608Metric_Pad1.05x0.95mm_HandSolder" V 3980 4950 50  0001 C CNN
 F 3 "~" H 4050 4950 50  0001 C CNN
 	1    4050 4950
@@
 F 0 "R32" H 4480 5704 50  0000 R CNN
 F 1 "1.6K" H 4480 5795 50  0000 R CNN
-F 2 "Resistor_SMD:R_0603_1608Metric" V 4480 5750 50  0001 C CNN
+F 2 "Resistor_SMD:R_0603_1608Metric_Pad1.05x0.95mm_HandSolder" V 4480 5750 50  0001 C CNN
 F 3 "~" H 4550 5750 50  0001 C CNN
 	1    4550 5750
@@
 F 0 "R33" V 4493 1000 50  0000 C CNN
 F 1 "4.7k" V 4584 1000 50  0000 C CNN
-F 2 "Resistor_SMD:R_0603_1608Metric" V 4630 1000 50  0001 C CNN
+F 2 "Resistor_SMD:R_0603_1608Metric_Pad1.05x0.95mm_HandSolder" V 4630 1000 50  0001 C CNN
 F 3 "~" H 4700 1000 50  0001 C CNN
 	1    4700 1000
@@
 F 0 "R30" H 3630 2004 50  0000 R CNN
 F 1 "470k" H 3630 2095 50  0000 R CNN
-F 2 "Resistor_SMD:R_0603_1608Metric" V 3630 2050 50  0001 C CNN
+F 2 "Resistor_SMD:R_0603_1608Metric_Pad1.05x0.95mm_HandSolder" V 3630 2050 50  0001 C CNN
 F 3 "~" H 3700 2050 50  0001 C CNN
 	1    3700 2050
@@
 F 0 "R28" H 3030 2004 50  0000 R CNN
 F 1 "2.7k" H 3030 2095 50  0000 R CNN
-F 2 "Resistor_SMD:R_0603_1608Metric" V 3030 2050 50  0001 C CNN
+F 2 "Resistor_SMD:R_0603_1608Metric_Pad1.05x0.95mm_HandSolder" V 3030 2050 50  0001 C CNN
 F 3 "~" H 3100 2050 50  0001 C CNN
 	1    3100 2050
@@
 F 0 "R26" V 2543 1500 50  0000 C CNN
 F 1 "100k" V 2634 1500 50  0000 C CNN
-F 2 "Resistor_SMD:R_0603_1608Metric" V 2680 1500 50  0001 C CNN
+F 2 "Resistor_SMD:R_0603_1608Metric_Pad1.05x0.95mm_HandSolder" V 2680 1500 50  0001 C CNN
 F 3 "~" H 2750 1500 50  0001 C CNN
 	1    2750 1500
@@
 F 0 "R40" H 10080 1754 50  0000 R CNN
 F 1 "100k" H 10080 1845 50  0000 R CNN
-F 2 "Resistor_SMD:R_0603_1608Metric" V 10080 1800 50  0001 C CNN
+F 2 "Resistor_SMD:R_0603_1608Metric_Pad1.05x0.95mm_HandSolder" V 10080 1800 50  0001 C CNN
 F 3 "~" H 10150 1800 50  0001 C CNN
 	1    10150 1800
@@
 F 0 "R21" V 1293 1500 50  0000 C CNN
 F 1 "100" V 1384 1500 50  0000 C CNN
-F 2 "Resistor_SMD:R_0603_1608Metric" V 1430 1500 50  0001 C CNN
+F 2 "Resistor_SMD:R_0603_1608Metric_Pad1.05x0.95mm_HandSolder" V 1430 1500 50  0001 C CNN
 F 3 "~" H 1500 1500 50  0001 C CNN
 	1    1500 1500
